File: pcb/6502v2/RAM+ROM.kicad_sch (KiCad schematic)
At the start: 2 parts

Commit message: Finally figured out the address decode logic, hopefully im done for now
Parts:
- removed U?: CY62256-70PC, Package_DIP:DIP-28_W15.24mm, symbol Memory_RAM:CY62256-70PC
Connections:
- net RAM_CS renamed RAM_~{CS}
Other:
- note removed: "todo: add another ram chip"
Changed lines of the file:
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@@
     (rev "2")
-  )
-  (text "todo: add another ram chip" (at 128.778 116.078 0)
-    (effects (font (size 1.27 1.27)) (justify left bottom))
   )
   (hierarchical_label "A1" (shape input) (at 81.28 69.85 180)
@@
     (effects (font (size 1.27 1.27)) (justify left))
   )
-  (hierarchical_label "RAM_CS" (shape input) (at 106.68 90.17 0)
+  (hierarchical_label "RAM_~{CS}" (shape input) (at 106.68 90.17 0)
     (effects (font (size 1.27 1.27)) (justify left))
   )
@@
     (effects (font (size 1.27 1.27)) (justify right))
   )
-  (symbol (lib_id "Memory_RAM:CY62256-70PC") (at 156.718 85.344 0) (unit 1)
-    (in_bom yes) (on_board yes) (fields_autoplaced)
-    (property "Reference" "U?" (id 0) (at 158.7374 59.944 0)
-      (effects (font (size 1.27 1.27)) (justify left))
-    )
-    (property "Value" "CY62256-70PC" (id 1) (at 158.7374 62.484 0)
-      (effects (font (size 1.27 1.27)) (justify left))
-    )
-    (property "Footprint" "Package_DIP:DIP-28_W15.24mm" (id 2) (at 156.718 87.884 0)
-      (effects (font (size 1.27 1.27)) hide)
-    )
-    (property "Datasheet" "https://ecee.colorado.edu/~mcclurel/Cypress_SRAM_CY62256.pdf" (id 3) (at 156.718 87.884 0)
-      (effects (font (size 1.27 1.27)) hide)
-    )
-    (pin "14")
-    (pin "28")
-    (pin "1")
-    (pin "10")
-    (pin "11")
-    (pin "12")
-    (pin "13")
-    (pin "15")
-    (pin "16")
-    (pin "17")
-    (pin "18")
-    (pin "19")
-    (pin "2")
-    (pin "20")
-    (pin "21")
-    (pin "22")
-    (pin "23")
-    (pin "24")
-    (pin "25")
-    (pin "26")
-    (pin "27")
-    (pin "3")
-    (pin "4")
-    (pin "5")
-    (pin "6")
-    (pin "7")
-    (pin "8")
-    (pin "9")
-  )
   (symbol (lib_id "power:+5V") (at 93.98 62.23 0) (unit 1)

Commit message: just working
Parts:
- gave numbers to parts that had none: 1
Changed lines of the file:
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@@
   (symbol (lib_id "power:+5V") (at 93.98 62.23 0) (unit 1)
     (in_bom yes) (on_board yes) (fields_autoplaced)
-    (property "Reference" "#PWR0103" (id 0) (at 93.98 66.04 0)
+    (property "Reference" "#PWR09" (id 0) (at 93.98 66.04 0)
       (effects (font (size 1.27 1.27)) hide)
     )
@@
   (symbol (lib_id "Memory_RAM:CY62256-70PC") (at 93.98 85.09 0) (unit 1)
     (in_bom yes) (on_board yes) (fields_autoplaced)
-    (property "Reference" "U?" (id 0) (at 95.9994 59.69 0)
+    (property "Reference" "U3" (id 0) (at 95.9994 59.69 0)
       (effects (font (size 1.27 1.27)) (justify left))
     )
@@
   (symbol (lib_id "power:GND") (at 93.98 107.95 0) (unit 1)
     (in_bom yes) (on_board yes) (fields_autoplaced)
-    (property "Reference" "#PWR0102" (id 0) (at 93.98 114.3 0)
+    (property "Reference" "#PWR010" (id 0) (at 93.98 114.3 0)
       (effects (font (size 1.27 1.27)) hide)
     )
