File: pcb/6502v2/ROM.kicad_sch (KiCad schematic)
At the start: 1 part

Commit message: just working
Parts:
- gave numbers to parts that had none: 1
Changed lines of the file:
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@@
   (symbol (lib_id "power:+5V") (at 134.62 104.14 0) (unit 1)
     (in_bom yes) (on_board yes) (fields_autoplaced)
-    (property "Reference" "#PWR?" (id 0) (at 134.62 107.95 0)
+    (property "Reference" "#PWR050" (id 0) (at 134.62 107.95 0)
       (effects (font (size 1.27 1.27)) hide)
     )
@@
   (symbol (lib_id "Memory_EEPROM:28C256") (at 153.67 86.36 0) (unit 1)
     (in_bom yes) (on_board yes) (fields_autoplaced)
-    (property "Reference" "U?" (id 0) (at 155.6894 55.88 0)
+    (property "Reference" "U9" (id 0) (at 155.6894 55.88 0)
       (effects (font (size 1.27 1.27)) (justify left))
     )
@@
   (symbol (lib_id "power:+5V") (at 153.67 55.88 0) (unit 1)
     (in_bom yes) (on_board yes) (fields_autoplaced)
-    (property "Reference" "#PWR?" (id 0) (at 153.67 59.69 0)
+    (property "Reference" "#PWR051" (id 0) (at 153.67 59.69 0)
       (effects (font (size 1.27 1.27)) hide)
     )
@@
   (symbol (lib_id "power:GND") (at 153.67 116.84 0) (unit 1)
     (in_bom yes) (on_board yes) (fields_autoplaced)
-    (property "Reference" "#PWR?" (id 0) (at 153.67 123.19 0)
+    (property "Reference" "#PWR052" (id 0) (at 153.67 123.19 0)
       (effects (font (size 1.27 1.27)) hide)
     )
@@
   (symbol (lib_id "power:GND") (at 130.81 106.68 0) (unit 1)
     (in_bom yes) (on_board yes) (fields_autoplaced)
-    (property "Reference" "#PWR?" (id 0) (at 130.81 113.03 0)
+    (property "Reference" "#PWR049" (id 0) (at 130.81 113.03 0)
       (effects (font (size 1.27 1.27)) hide)
     )
