File: pcb/6502v2/6502v2.kicad_sch (KiCad schematic)
At the start: 70 parts, among them J1 Barrel_Jack, J2 I/O, J3 I/O, SW1 SW_Push, U1 CY62256-70PC, U2 W65C22NxP, U3 28C256, U4 74HC00, U5 W65C02SxP, X1 DGOF5S3

Commit message: Changed stufffs
Parts:
- removed C1, C2, C3: 10uf, Capacitor_SMD:C_0805_2012Metric, symbol Device:C_Small
- removed C4: 10uf, Resistor_SMD:R_0805_2012Metric, symbol Device:C_Small
- removed D1, D12, D14, D16, D3, D5, D7, D9: Blu, Resistor_SMD:R_0805_2012Metric, symbol Device:LED_Small
- removed D10, D13, D15, D17, D18, D19, D2, D20, D22, D23, D24, D25, D26, D4, D6, D8: Red, Resistor_SMD:R_0805_2012Metric, symbol Device:LED_Small
- removed D11: Green, Resistor_SMD:R_0805_2012Metric, symbol Device:LED_Small
- removed D21: Yellow, Resistor_SMD:R_0805_2012Metric, symbol Device:LED_Small
- removed J1: Barrel_Jack, Connector_BarrelJack:BarrelJack_GCT_DCJ200-10-A_Horizontal, symbol Connector:Barrel_Jack
- removed J2, J3: I/O, Connector_PinSocket_2.54mm:PinSocket_1x08_P2.54mm_Vertical, symbol Connector_Generic:Conn_01x08
- removed J?: Conn_01x02, symbol Connector_Generic:Conn_01x02
- removed R1, R10, R11, R12, R13, R14, R15, R16, R17, R18, R19, R2, R20, R21, R22, R23, R24, R25, R26, R27, R29, R3, R4, R5, R6, R7, R8, R9: 220, Resistor_SMD:R_0805_2012Metric, symbol Device:R_Small
- removed R28: 1k, Resistor_SMD:R_0805_2012Metric, symbol Device:R_Small
- removed SW1: SW_Push, Button_Switch_SMD:SW_SPST_TL3342, symbol Switch:SW_Push
- removed U1: CY62256-70PC, Package_DIP:DIP-28_W15.24mm, symbol Memory_RAM:CY62256-70PC
- removed U2: W65C22NxP, Package_DIP:DIP-40_W15.24mm, symbol 65xx:W65C22NxP
- removed U5: W65C02SxP, Package_DIP:DIP-40_W15.24mm, symbol 65xx:W65C02SxP
- added J?: Power, symbol Connector:Screw_Terminal_01x02
Connections:
- net CLK renamed Clk
- new net Power Input/5V power: J?.1 (Pin_1)
- new net Power Input/GND: J?.2 (Pin_2)
- no-connect marks 2 -> 0
Other:
- added sheet Address and Data LEDs (dataLeds.kicad_sch)
- added sheet CPU (CPU.kicad_sch)
- added sheet Power Input (Power.kicad_sch)
- added sheet RAM and ROM (RAM+ROM.kicad_sch)
- added sheet VIA (via.kicad_sch)
- note added: "A"
- note added: "ROM"
- note removed: "Barrel Jack and power indicator led"
- note removed: "Debug leds"
- note removed: "I/O header"
- note removed: "I/O interface"
- note removed: "Main processor connections"
- note removed: "One per ic"
- note removed: "Power Filtering"
- note removed: "Storage eeprom"
- title: (none) -> 6502 Computer
- moved on the sheet: X1

Commit message: UART more like u r dumb
Other:
- sheet RAM and ROM renamed RAM
- added sheet Serial (Serial.kicad_sch)
- sheet VIA ports: added LCD C22 Enable, LCD C22 ~{Enable}, ~{IRQ}; removed none

Commit message: Finally figured out the address decode logic, hopefully im done for now
Parts:
- removed U3: 28C256, Package_DIP:DIP-28_W15.24mm, symbol Memory_EEPROM:28C256
- added U?: 74HC238, symbol 74xx:74HC238
Connections:
- net +5V: now also U?.16 (VCC), U?.6 (E3)
- net A4: now also U?.1 (A0)
- net A5: now also U?.2 (A1)
- net A6: now also U?.3 (A2)
- net C22 Enable: now also U?.14 (Y1); no longer U4.8
- net GND: now also U?.4 (~{E1}), U?.5 (~{E2}), U?.8 (GND)
- net Inv_A15 renamed ~{A15}
- net RAM_CS renamed RAM ~{CS}
- new net I/O ~{Enable}: U4.8
- new net LCD C22 Enable: U?.13 (Y2)
- new net Serial ~{Enable}: U?.11 (Y4)
- no-connect marks 0 -> 3
Other:
- added sheet ROM (ROM.kicad_sch)
- sheet RAM ports: added RAM_~{CS}; removed RAM_CS
- sheet Serial ports: added A0, A1, Serial Enable, Serial ~{Enable}; removed none
- note removed: "ROM"
- moved on the sheet: U4A, U4B, U4C, U4D

Commit message: just working
Parts:
- J1: renamed from J?; footprint (none) -> TerminalBlock:TerminalBlock_bornier-2_P5.08mm
- U2: renamed from U?; footprint (none) -> Package_DIP:DIP-16_W7.62mm
- renumbered U4 to U1

Commit message: Laying out chips
Connections:
- net Serial ~{Enable} is gone; now on net Serial Enable: U2.11 (Y4)
Changed lines of the file:
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@@
     (effects (font (size 1.27 1.27)) (justify left bottom))
+  )
+  (label "Serial Enable" (at 189.992 147.828 180)
+    (effects (font (size 1.27 1.27)) (justify right bottom))
   )
   (label "D7" (at 116.332 70.612 180)
@@
     (effects (font (size 1.27 1.27)) (justify left bottom))
   )
-  (label "Serial ~{Enable}" (at 189.992 147.828 180)
-    (effects (font (size 1.27 1.27)) (justify right bottom))
-  )
   (label "D7" (at 160.274 38.1 180)

Commit message: Tidying up schematic
Other:
- note added: "Debug LEDs"
- note added: "GPIO"
- note added: "Main CPU and clock"
- note added: "Power"
- note added: "RAM and ROM"
- note added: "Serial Interface"
- moved on the sheet: U1A, U1B, U1C, U1D, U1E, U2, X1
