File: pcb/6502v2/dataLeds.kicad_sch (KiCad schematic)
At the start: 50 parts

Commit message: just working
Parts:
- gave numbers to parts that had none: 50

Commit message: Tidying up schematic
Other:
- note added: "Due to lack of space, the address LEDs were not included on the final PBC"
Changed lines of the file:
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@@
     (stroke (width 0) (type default) (color 0 0 0 0))
+  )
+  (text "Due to lack of space, the address \nLEDs were not included on the final PBC"
+    (at 126.238 119.888 0)
+    (effects (font (size 1.27 1.27)) (justify left bottom))
   )
   (text "LEDs" (at 171.958 82.804 180)
