File: pcb/6502v2/6502v2.kicad_pcb (KiCad board)
At the start: 4 copper layers, 102 x 102 mm, 64 parts, among them J1 Power, J5 Interup Pins, J8 Interup Pins, J9 DB9_Female, U9 28C256

Commit message: Finishing up
Other:
- board text removed: "Anjali <333"
Changed lines of the file:
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@@
       (drillshape 0)
       (scaleselection 1)
-      (outputdirectory "../gerbers/")
+      (outputdirectory "../../gerbers/")
     )
   )
@@
     (effects (font (size 1 1) (thickness 0.15)))
   )
-  (gr_text "Anjali <333\n" (at 46.45 124.1) (layer "F.SilkS")
-    (effects (font (size 0.5 0.5) (thickness 0.125)))
-  )
   (gr_text "LCD Int Pins\n" (at 102.65 92.35 90) (layer "F.SilkS")

Commit message: Removed burried VIAs because jlc cant produce them
Routing:
- net /A12: track 85.5 -> 86.3 mm
Other:
- board text added: "Anjali <33"

Commit message: Fixed mirrored footprints, updated readme
Parts:
- removed D1: Green, Resistor_SMD:R_0805_2012Metric
- removed R3: 220, Resistor_SMD:R_0805_2012Metric
- J7: renamed from LCD Header
- Y1: renamed from 1.8432 Mh
- renumbered Fuse to F1, 5v to J2, NMI to J3, GPIO to J4, GPIO to J6, Reset to SW1, 74HC00 to U1, 74HC238 to U2, RAM to U3, 65C02 to U4, 65C22 to U5, 65C22 to U6, MAX232 to U7, 65C51 to U8, 1Mh to X1
Connections:
- J7 pad 10: /VIA/LCD PB0 -> /VIA/LCD PB3
- J7 pad 11: /VIA/LCD PA7 -> /VIA/LCD PB4
- J7 pad 12: /VIA/LCD PA6 -> /VIA/LCD PB5
- J7 pad 13: /VIA/LCD PA5 -> /VIA/LCD PB6
- J7 pad 14: Net-(J7-Pad14) -> /VIA/LCD PB7
- J7 pad 3: /VIA/LCD PB7 -> Net-(J7-Pad3)
- J7 pad 4: /VIA/LCD PB6 -> /VIA/LCD PA5
- J7 pad 5: /VIA/LCD PB5 -> /VIA/LCD PA6
- J7 pad 6: /VIA/LCD PB4 -> /VIA/LCD PA7
- J7 pad 7: /VIA/LCD PB3 -> /VIA/LCD PB0
- J7 pad 8: /VIA/LCD PB2 -> /VIA/LCD PB1
- J7 pad 9: /VIA/LCD PB1 -> /VIA/LCD PB2
- R32 pad 1: Net-(J7-Pad14) -> Net-(J7-Pad3)
Routing:
- net /VIA/LCD PB4: track 13.9 -> 58.6 mm
- net /VIA/LCD PB3: track 13.9 -> 55.9 mm
- net /VIA/LCD PB5: track 13.9 -> 51.9 mm
- net /VIA/LCD PB6: track 13.9 -> 47.4 mm
- net Net-(J7-Pad3): track 0.00 -> 30.3 mm, vias 0 -> 1
- net /VIA/LCD PB7: track 13.9 -> 42.8 mm
- net /VIA/LCD PB0: track 13.9 -> 42.7 mm
- net /VIA/LCD PA7: track 13.9 -> 37.7 mm
- net /VIA/LCD PA6: track 13.9 -> 31.6 mm
- net /VIA/LCD PA5: track 13.9 -> 27.3 mm
- net /A2: track 152.4 -> 164.1 mm
- net /A3: track 195.4 -> 205.6 mm
- net /VIA/LCD PB2: track 13.9 -> 20.4 mm
- net Net-(J7-Pad14): track 3.20 -> 0.00 mm
- net /VIA/LCD PB1: track 13.9 -> 13.1 mm
