File: pcb/6502v2/via.kicad_sch (KiCad schematic)
At the start: 3 parts

Commit message: UART more like u r dumb
Parts:
- added J? (x2): Interup Pins, symbol Connector_Generic:Conn_01x04
- added J? (x2): I/O, Connector_PinSocket_2.54mm:PinSocket_1x08_P2.54mm_Vertical, symbol Connector_Generic:Conn_01x08
- added J?: LDC, symbol Connector_Generic:Conn_01x16
- added R?: R_Small, symbol Device:R_Small
- added U?: W65C22NxP, Package_DIP:DIP-40_W15.24mm, symbol 65xx:W65C22NxP
Connections:
- net +5V: now also J?.15 (Pin_15), J?.2 (Pin_2), U?.20 (VCC)
- net A0: now also U?.38 (RS0)
- net A1: now also U?.37 (RS1)
- net A2: now also U?.36 (RS2)
- net A3: now also U?.35 (RS3)
- net CLK: now also U?.25 (ϕ2)
- net D0: now also U?.33 (D0)
- net D1: now also U?.32 (D1)
- net D2: now also U?.31 (D2)
- net D3: now also U?.30 (D3)
- net D4: now also U?.29 (D4)
- net D5: now also U?.28 (D5)
- net D6: now also U?.27 (D6)
- net D7: now also U?.26 (D7)
- net GND: now also J?.1 (Pin_1), J?.16 (Pin_16), R?.2, U?.1 (VSS)
- net RESET: now also U?.34 (~{RES})
- net R/W: now also U?.22 (R/~{W})
- net CB1: now reaches U?.18 (CB1)
- net CB1: now also J?.3 (Pin_3)
- net CB2: now reaches U?.19 (CB2)
- net CB2: now also J?.4 (Pin_4)
- net ~{IRQ}: now reaches U?.21 (~{IRQ})
- net CA2: now reaches U?.39 (CA2)
- net CA2: now also J?.2 (Pin_2)
- net CA1: now reaches U?.40 (CA1)
- net CA1: now also J?.1 (Pin_1)
- new net: J?.14 (Pin_14), R?.1
- new net LCD C22 Enable: U?.24 (CS1)
- new net LCD C22 ~{Enable}: U?.23 (~{CS2})
- new net LCD CA1: J?.1 (Pin_1), U?.40 (CA1)
- new net LCD CA2: J?.2 (Pin_2), U?.39 (CA2)
- new net LCD CB1: J?.3 (Pin_3), U?.18 (CB1)
- new net LCD CB2: J?.4 (Pin_4), U?.19 (CB2)
- new net LCD PA0: J?.8 (Pin_8), U?.2 (PA0)
- new net LCD PA1: J?.7 (Pin_7), U?.3 (PA1)
- new net LCD PA2: J?.6 (Pin_6), U?.4 (PA2)
- new net LCD PA3: J?.5 (Pin_5), U?.5 (PA3)
- new net LCD PA4: J?.4 (Pin_4), U?.6 (PA4)
- new net LCD PA5: J?.13 (Pin_13), J?.3 (Pin_3), U?.7 (PA5)
- new net LCD PA6: J?.12 (Pin_12), J?.2 (Pin_2), U?.8 (PA6)
- new net LCD PA7: J?.1 (Pin_1), J?.11 (Pin_11), U?.9 (PA7)
- new net LCD PB0: J?.10 (Pin_10), J?.8 (Pin_8), U?.10 (PB0)
- new net LCD PB1: J?.7 (Pin_7), J?.9 (Pin_9), U?.11 (PB1)
- new net LCD PB2: J?.6 (Pin_6), J?.8 (Pin_8), U?.12 (PB2)
- new net LCD PB3: J?.5 (Pin_5), J?.7 (Pin_7), U?.13 (PB3)
- new net LCD PB4: J?.4 (Pin_4), J?.6 (Pin_6), U?.14 (PB4)
- new net LCD PB5: J?.3 (Pin_3), J?.5 (Pin_5), U?.15 (PB5)
- new net LCD PB6: J?.2 (Pin_2), J?.4 (Pin_4), U?.16 (PB6)
- new net LCD PB7: J?.1 (Pin_1), J?.3 (Pin_3), U?.17 (PB7)
- no-connect marks 0 -> 1
Other:
- note added: "GPIO VIA"
- note added: "LCD Display VIA"

Commit message: just working
Parts:
- J10, J6: renamed from J?; footprint (none) -> Connector_PinHeader_2.54mm:PinHeader_1x04_P2.54mm_Vertical
- J9: renamed from J?; footprint (none) -> Connector_PinSocket_2.54mm:PinSocket_1x16_P2.54mm_Vertical
- R32: renamed from R?; footprint (none) -> Resistor_SMD:R_0805_2012Metric
- gave numbers to parts that had none: 6
Changed lines of the file:
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@@
   (symbol (lib_id "Connector_Generic:Conn_01x08") (at 122.936 66.04 0) (unit 1)
     (in_bom yes) (on_board yes) (fields_autoplaced)
-    (property "Reference" "J?" (id 0) (at 125.476 66.0399 0)
+    (property "Reference" "J7" (id 0) (at 125.476 66.0399 0)
       (effects (font (size 1.27 1.27)) (justify left))
     )
@@
   (symbol (lib_id "Connector_Generic:Conn_01x04") (at 102.87 87.122 0) (unit 1)
     (in_bom yes) (on_board yes) (fields_autoplaced)
-    (property "Reference" "J?" (id 0) (at 105.41 87.1219 0)
+    (property "Reference" "J6" (id 0) (at 105.41 87.1219 0)
       (effects (font (size 1.27 1.27)) (justify left))
     )
@@
       (effects (font (size 1.27 1.27)) (justify left))
     )
-    (property "Footprint" "" (id 2) (at 102.87 87.122 0)
+    (property "Footprint" "Connector_PinHeader_2.54mm:PinHeader_1x04_P2.54mm_Vertical" (id 2) (at 102.87 87.122 0)
       (effects (font (size 1.27 1.27)) hide)
     )
@@
   (symbol (lib_id "power:GND") (at 162.306 133.35 0) (unit 1)
     (in_bom yes) (on_board yes) (fields_autoplaced)
-    (property "Reference" "#PWR0101" (id 0) (at 162.306 139.7 0)
+    (property "Reference" "#PWR034" (id 0) (at 162.306 139.7 0)
       (effects (font (size 1.27 1.27)) hide)
     )
@@
   (symbol (lib_id "65xx:W65C22NxP") (at 162.306 95.25 0) (unit 1)
     (in_bom yes) (on_board yes) (fields_autoplaced)
-    (property "Reference" "U?" (id 0) (at 164.3254 58.42 0)
+    (property "Reference" "U5" (id 0) (at 164.3254 58.42 0)
       (effects (font (size 1.27 1.27)) (justify left))
     )
@@
   (symbol (lib_id "power:+5V") (at 267.462 150.622 0) (unit 1)
     (in_bom yes) (on_board yes) (fields_autoplaced)
-    (property "Reference" "#PWR0136" (id 0) (at 267.462 154.432 0)
+    (property "Reference" "#PWR040" (id 0) (at 267.462 154.432 0)
       (effects (font (size 1.27 1.27)) hide)
     )
@@
   (symbol (lib_id "Connector_Generic:Conn_01x08") (at 102.616 66.04 0) (unit 1)
     (in_bom yes) (on_board yes)
-    (property "Reference" "J?" (id 0) (at 105.156 66.0399 0)
+    (property "Reference" "J5" (id 0) (at 105.156 66.0399 0)
       (effects (font (size 1.27 1.27)) (justify left))
     )
@@
   (symbol (lib_id "power:GND") (at 274.066 150.622 0) (unit 1)
     (in_bom yes) (on_board yes) (fields_autoplaced)
-    (property "Reference" "#PWR0137" (id 0) (at 274.066 156.972 0)
+    (property "Reference" "#PWR041" (id 0) (at 274.066 156.972 0)
       (effects (font (size 1.27 1.27)) hide)
     )
@@
   (symbol (lib_id "65xx:W65C22NxP") (at 229.87 97.536 0) (unit 1)
     (in_bom yes) (on_board yes) (fields_autoplaced)
-    (property "Reference" "U?" (id 0) (at 231.8894 60.706 0)
+    (property "Reference" "U6" (id 0) (at 231.8894 60.706 0)
       (effects (font (size 1.27 1.27)) (justify left))
     )
@@
   (symbol (lib_id "Connector_Generic:Conn_01x08") (at 268.732 30.988 180) (unit 1)
     (in_bom yes) (on_board yes) (fields_autoplaced)
-    (property "Reference" "J?" (id 0) (at 268.732 13.97 0))
+    (property "Reference" "J11" (id 0) (at 268.732 13.97 0))
     (property "Value" "I/O" (id 1) (at 268.732 16.51 0))
     (property "Footprint" "Connector_PinSocket_2.54mm:PinSocket_1x08_P2.54mm_Vertical" (id 2) (at 268.732 30.988 0)
@@
   (symbol (lib_id "power:+5V") (at 234.442 150.368 0) (unit 1)
     (in_bom yes) (on_board yes) (fields_autoplaced)
-    (property "Reference" "#PWR0138" (id 0) (at 234.442 154.178 0)
+    (property "Reference" "#PWR038" (id 0) (at 234.442 154.178 0)
       (effects (font (size 1.27 1.27)) hide)
     )
@@
   (symbol (lib_id "Device:R_Small") (at 236.982 147.066 180) (unit 1)
     (in_bom yes) (on_board yes)
-    (property "Reference" "R?" (id 0) (at 234.188 141.224 0)
+    (property "Reference" "R32" (id 0) (at 234.188 141.224 0)
       (effects (font (size 1.27 1.27)) (justify right))
     )
@@
       (effects (font (size 1.27 1.27)) (justify right))
     )
-    (property "Footprint" "" (id 2) (at 236.982 147.066 0)
+    (property "Footprint" "Resistor_SMD:R_0805_2012Metric" (id 2) (at 236.982 147.066 0)
       (effects (font (size 1.27 1.27)) hide)
     )
@@
   (symbol (lib_id "Connector_Generic:Conn_01x04") (at 268.224 52.07 0) (unit 1)
     (in_bom yes) (on_board yes) (fields_autoplaced)
-    (property "Reference" "J?" (id 0) (at 270.764 52.0699 0)
+    (property "Reference" "J10" (id 0) (at 270.764 52.0699 0)
       (effects (font (size 1.27 1.27)) (justify left))
     )
@@
       (effects (font (size 1.27 1.27)) (justify left))
     )
-    (property "Footprint" "" (id 2) (at 268.224 52.07 0)
+    (property "Footprint" "Connector_PinHeader_2.54mm:PinHeader_1x04_P2.54mm_Vertical" (id 2) (at 268.224 52.07 0)
       (effects (font (size 1.27 1.27)) hide)
     )
@@
   (symbol (lib_id "power:GND") (at 239.776 140.462 0) (unit 1)
     (in_bom yes) (on_board yes)
-    (property "Reference" "#PWR0139" (id 0) (at 239.776 146.812 0)
+    (property "Reference" "#PWR039" (id 0) (at 239.776 146.812 0)
       (effects (font (size 1.27 1.27)) hide)
     )
@@
   (symbol (lib_id "Connector_Generic:Conn_01x08") (at 248.412 30.988 180) (unit 1)
     (in_bom yes) (on_board yes)
-    (property "Reference" "J?" (id 0) (at 245.872 30.9881 0)
+    (property "Reference" "J8" (id 0) (at 245.872 30.9881 0)
       (effects (font (size 1.27 1.27)) (justify left))
     )
@@
   (symbol (lib_id "power:+5V") (at 229.87 59.182 0) (unit 1)
     (in_bom yes) (on_board yes) (fields_autoplaced)
-    (property "Reference" "#PWR0141" (id 0) (at 229.87 62.992 0)
+    (property "Reference" "#PWR036" (id 0) (at 229.87 62.992 0)
       (effects (font (size 1.27 1.27)) hide)
     )
@@
   (symbol (lib_id "power:+5V") (at 162.306 57.15 0) (unit 1)
     (in_bom yes) (on_board yes) (fields_autoplaced)
-    (property "Reference" "#PWR0140" (id 0) (at 162.306 60.96 0)
+    (property "Reference" "#PWR033" (id 0) (at 162.306 60.96 0)
       (effects (font (size 1.27 1.27)) hide)
     )
@@
   (symbol (lib_id "Connector_Generic:Conn_01x16") (at 252.222 158.242 270) (unit 1)
     (in_bom yes) (on_board yes) (fields_autoplaced)
-    (property "Reference" "J?" (id 0) (at 250.952 162.56 90))
+    (property "Reference" "J9" (id 0) (at 250.952 162.56 90))
     (property "Value" "LDC" (id 1) (at 250.952 165.1 90))
-    (property "Footprint" "" (id 2) (at 252.222 158.242 0)
+    (property "Footprint" "Connector_PinSocket_2.54mm:PinSocket_1x16_P2.54mm_Vertical" (id 2) (at 252.222 158.242 0)
       (effects (font (size 1.27 1.27)) hide)
     )
@@
   (symbol (lib_id "power:GND") (at 226.06 150.368 0) (unit 1)
     (in_bom yes) (on_board yes) (fields_autoplaced)
-    (property "Reference" "#PWR0127" (id 0) (at 226.06 156.718 0)
+    (property "Reference" "#PWR035" (id 0) (at 226.06 156.718 0)
       (effects (font (size 1.27 1.27)) hide)
     )
@@
   (symbol (lib_id "power:GND") (at 229.87 135.89 0) (unit 1)
     (in_bom yes) (on_board yes) (fields_autoplaced)
-    (property "Reference" "#PWR0135" (id 0) (at 229.87 142.24 0)
-      (effects (font (size 1.27 1.27)) hide)
-    )
+    (property "Reference" "#PWR037" (id 0) (at 229.87 142.24 0)
+      (effects (font (size 1.27 1.27)) hide)
+    )

Commit message: Yo yo yo i make the bord 102 by 102 cause jlc pricing
Parts:
- removed J11, J5, J7, J8: I/O, Connector_PinSocket_2.54mm:PinSocket_1x08_P2.54mm_Vertical, symbol Connector_Generic:Conn_01x08
- added J5, J7: I/O, Connector_PinSocket_2.54mm:PinSocket_1x16_P2.54mm_Vertical, symbol Connector_Generic:Conn_01x16
- renumbered J9 to J8, J10 to J9
Connections:
- net LCD PA0: now also J7.16 (Pin_16)
- net LCD PA1: now also J7.15 (Pin_15)
- net LCD PA2: now also J7.14 (Pin_14)
- net LCD PA3: now also J7.13 (Pin_13)
- net LCD PA4: now also J7.12 (Pin_12)
- net LCD PA5: now also J7.11 (Pin_11)
- net LCD PA6: now also J7.10 (Pin_10)
- net LCD PA7: now also J7.9 (Pin_9)
- net LCD PB0: now also J7.8 (Pin_8)
- net LCD PB1: now also J7.7 (Pin_7)
- net LCD PB2: now also J7.6 (Pin_6)
- net LCD PB3: now also J7.5 (Pin_5)
- net LCD PB4: now also J7.4 (Pin_4)
- net LCD PB5: now also J7.3 (Pin_3)
- net LCD PB6: now also J7.2 (Pin_2)
- net LCD PB7: now also J7.1 (Pin_1)
- net PA0: now also J5.1 (Pin_1)
- net PA1: now also J5.2 (Pin_2)
- net PA2: now also J5.3 (Pin_3)
- net PA3: now also J5.4 (Pin_4)
- net PA4: now also J5.5 (Pin_5)
- net PA5: now also J5.6 (Pin_6)
- net PA6: now also J5.7 (Pin_7)
- net PA7: now also J5.8 (Pin_8)
- net PB0: now also J5.9 (Pin_9)
- net PB1: now also J5.10 (Pin_10)
- net PB2: now also J5.11 (Pin_11)
- net PB3: now also J5.12 (Pin_12)
- net PB4: now also J5.13 (Pin_13)
- net PB5: now also J5.14 (Pin_14)
- net PB6: now also J5.15 (Pin_15)
- net PB7: now also J5.16 (Pin_16)

Commit message: First pass at routing done, now comes double checking everything
Parts:
- renumbered J5 to J4, J6 to J5, J7 to J6, J8 to J7, J9 to J8
Changed lines of the file:
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@@
   (symbol (lib_id "Connector_Generic:Conn_01x04") (at 102.87 87.122 0) (unit 1)
     (in_bom yes) (on_board yes) (fields_autoplaced)
-    (property "Reference" "J6" (id 0) (at 105.41 87.1219 0)
+    (property "Reference" "J5" (id 0) (at 105.41 87.1219 0)
       (effects (font (size 1.27 1.27)) (justify left))
     )
@@
   (symbol (lib_id "power:GND") (at 162.306 133.35 0) (unit 1)
     (in_bom yes) (on_board yes) (fields_autoplaced)
-    (property "Reference" "#PWR036" (id 0) (at 162.306 139.7 0)
+    (property "Reference" "#PWR039" (id 0) (at 162.306 139.7 0)
       (effects (font (size 1.27 1.27)) hide)
     )
@@
   (symbol (lib_id "power:+5V") (at 267.462 150.622 0) (unit 1)
     (in_bom yes) (on_board yes) (fields_autoplaced)
-    (property "Reference" "#PWR042" (id 0) (at 267.462 154.432 0)
+    (property "Reference" "#PWR045" (id 0) (at 267.462 154.432 0)
       (effects (font (size 1.27 1.27)) hide)
     )
@@
   (symbol (lib_id "power:GND") (at 274.066 150.622 0) (unit 1)
     (in_bom yes) (on_board yes) (fields_autoplaced)
-    (property "Reference" "#PWR043" (id 0) (at 274.066 156.972 0)
+    (property "Reference" "#PWR046" (id 0) (at 274.066 156.972 0)
       (effects (font (size 1.27 1.27)) hide)
     )
@@
   (symbol (lib_id "power:+5V") (at 234.442 150.368 0) (unit 1)
     (in_bom yes) (on_board yes) (fields_autoplaced)
-    (property "Reference" "#PWR040" (id 0) (at 234.442 154.178 0)
+    (property "Reference" "#PWR043" (id 0) (at 234.442 154.178 0)
       (effects (font (size 1.27 1.27)) hide)
     )
@@
   (symbol (lib_id "Connector_Generic:Conn_01x04") (at 268.224 52.07 0) (unit 1)
     (in_bom yes) (on_board yes) (fields_autoplaced)
-    (property "Reference" "J9" (id 0) (at 270.764 52.0699 0)
+    (property "Reference" "J8" (id 0) (at 270.764 52.0699 0)
       (effects (font (size 1.27 1.27)) (justify left))
     )
@@
   (symbol (lib_id "power:GND") (at 239.776 140.462 0) (unit 1)
     (in_bom yes) (on_board yes)
-    (property "Reference" "#PWR041" (id 0) (at 239.776 146.812 0)
+    (property "Reference" "#PWR044" (id 0) (at 239.776 146.812 0)
       (effects (font (size 1.27 1.27)) hide)
     )
@@
   (symbol (lib_id "Connector_Generic:Conn_01x16") (at 235.966 32.258 180) (unit 1)
     (in_bom yes) (on_board yes) (fields_autoplaced)
-    (property "Reference" "J7" (id 0) (at 235.966 5.588 0))
+    (property "Reference" "J6" (id 0) (at 235.966 5.588 0))
     (property "Value" "I/O" (id 1) (at 235.966 8.128 0))
     (property "Footprint" "Connector_PinSocket_2.54mm:PinSocket_1x16_P2.54mm_Vertical" (id 2) (at 235.966 32.258 0)
@@
   (symbol (lib_id "Connector_Generic:Conn_01x16") (at 72.644 65.024 0) (unit 1)
     (in_bom yes) (on_board yes) (fields_autoplaced)
-    (property "Reference" "J5" (id 0) (at 74.93 65.0239 0)
+    (property "Reference" "J4" (id 0) (at 74.93 65.0239 0)
       (effects (font (size 1.27 1.27)) (justify left))
     )
@@
   (symbol (lib_id "power:+5V") (at 229.87 59.182 0) (unit 1)
     (in_bom yes) (on_board yes) (fields_autoplaced)
-    (property "Reference" "#PWR038" (id 0) (at 229.87 62.992 0)
+    (property "Reference" "#PWR041" (id 0) (at 229.87 62.992 0)
       (effects (font (size 1.27 1.27)) hide)
     )
@@
   (symbol (lib_id "power:+5V") (at 162.306 57.15 0) (unit 1)
     (in_bom yes) (on_board yes) (fields_autoplaced)
-    (property "Reference" "#PWR035" (id 0) (at 162.306 60.96 0)
+    (property "Reference" "#PWR038" (id 0) (at 162.306 60.96 0)
       (effects (font (size 1.27 1.27)) hide)
     )
@@
   (symbol (lib_id "Connector_Generic:Conn_01x16") (at 252.222 158.242 270) (unit 1)
     (in_bom yes) (on_board yes) (fields_autoplaced)
-    (property "Reference" "J8" (id 0) (at 250.952 162.56 90))
+    (property "Reference" "J7" (id 0) (at 250.952 162.56 90))
     (property "Value" "LDC" (id 1) (at 250.952 165.1 90))
     (property "Footprint" "Connector_PinSocket_2.54mm:PinSocket_1x16_P2.54mm_Vertical" (id 2) (at 252.222 158.242 0)
@@
   (symbol (lib_id "power:GND") (at 226.06 150.368 0) (unit 1)
     (in_bom yes) (on_board yes) (fields_autoplaced)
-    (property "Reference" "#PWR037" (id 0) (at 226.06 156.718 0)
+    (property "Reference" "#PWR040" (id 0) (at 226.06 156.718 0)
       (effects (font (size 1.27 1.27)) hide)
     )
@@
   (symbol (lib_id "power:GND") (at 229.87 135.89 0) (unit 1)
     (in_bom yes) (on_board yes) (fields_autoplaced)
-    (property "Reference" "#PWR039" (id 0) (at 229.87 142.24 0)
-      (effects (font (size 1.27 1.27)) hide)
-    )
+    (property "Reference" "#PWR042" (id 0) (at 229.87 142.24 0)
+      (effects (font (size 1.27 1.27)) hide)
+    )
